File: kicad/ITX-Llama.kicad_sch (KiCad schematic)
At the start: 421 parts, among them J1 ATX_POWER, J10 SATA, J11 SPEAKER, J12 MSD, J14 AUDIO, J15 KBC, J16 KBD, J17 USB_ETH, J18 USB_HID, J19 HID_POWER, J2 MICRO_SD, J20 FAN1, J21 FAN2, J22 GAMEPORT, J23 WAVETABLE, J24 PI_ZERO2, J25 POWER, J26 LEFT, J27 RIGHT, J28 COM2_TTL, J29 PI_2/3/4, J3 FRONT_PANEL, J30 FAN3, J31 FAN1_VDD, J32 FAN2_VDD, J33 FAN3_VDD, J34 CD_IN, J35 D1_MINI, J36 ESP_POWER, J38 J_TOSLINK_ZGY133T10, J39 LINE_L, J4 PS/2, J40 LINE_R, J41 EXT_SYNTH, J42 PI_I2C, J43 I2C, J46 RP_DEBUG, J5 AGP_3.3V, J6 CLICK_VOL, J7 MSC, J8 COM1, J9 INT_SPKR_VOL, P1 P_SOM-128-EX, Q1 NPN, Q10 Q_NMOS_GDS, Q11 Q_NMOS_GDS, Q2 NPN, Q3 NPN, Q4 NPN, Q5 NPN, Q6 NPN, Q7 NPN, Q8 Q_NMOS_GDS, Q9 Q_NMOS_GDS, SW1 CH559_PRG, SW1 POWER, SW2 RESET, T1 Pulse_H1102NL, U1 MAX16054, U10 U_MIC5219-3.3YM5, U11 EMC2303, U12 PCM5102A, U13 U_MIC5219-3.3YM5, U14 U_MIC5219-3.3YM5, U15 W25Q32JVSS, U16 U_74LVC1G126, U17 U_RP2040, U2 U_74LVC1G04, U3 U_CS4237B-KQ, U4 GD75232, U5 U_MC33078, U6 PI7C9X118SL, U7 AP7165, U8 U_MIC5219-3.3YM5, U9 U_ATTINY84A, X1 16.9344MHz, X2 12MHz

Commit message: Update Kicad project for rev.F
Parts:
- removed FB8, FB9: 70Ω@100MHz, llama_shared:R_0603_1608Metric, symbol llama_shared:FB
- removed J25: POWER, llama_shared:P_CONN_01X03, symbol Connector_Generic:Conn_01x03
- added J13: MT32-PI-GND, llama_shared:P_CONN_01X05, symbol llama_shared:P_MT32PI_GND
- added LOGO2: RD_Logo, tinyllama:LOGO_retrodreams, symbol llama_shared:Llama_logo
- added R122, R123: 27, llama_shared:R_0402_1005Metric, symbol llama_shared:R
- BT1: symbol tinyllama_shared:BT -> llama_shared:BT
- C27: LCSC (none) -> C140782
- J1: LCSC C114125 -> C114088
- J42: value PI_I2C -> MT32-PI; footprint llama_shared:P_CONN_01X04 -> llama_shared:P_CONN_01X09; symbol llama_shared:P_091OLED -> llama_shared:P_MT32PI
- LOGO1: footprint llama_shared:LLAMA_LOGO -> llama_shared:LOGO_llama
- Q10, Q11, Q8, Q9: LCSC C255592 -> C5224263
- U3: LCSC (none) -> C9900149464
Connections:
- net VCC_3V3_AGP is gone; now on net +3.3V: C129.2, C130.2, C131.2, C159.1, C162.2, C164.2, C165.2, C166.2, C167.1, C168.1, C173.1, C61.1, C62.1, C63.2, J5.A16 (VCC_3.3V), J5.A28 (VCC_3.3V), J5.A45 (VCC_3.3V), J5.A9 (VCC_3.3V), J5.B16 (VCC_3.3V), J5.B28 (VCC_3.3V), J5.B45 (VCC_3.3V), J5.B9 (VCC_3.3V)
- net VCC_VIO_AGP is gone; now on net +3.3V: C169.1, C170.1, C38.2, C39.2, C40.2, C41.2, C42.2, C43.1, C44.1, C45.1, C46.1, C47.1, C53.1, C54.2, C56.2, C57.2, C58.2, C59.2, C60.2, J5.A34 (Vddq3.3), J5.A40 (Vddq3.3), J5.A52 (Vddq3.3), J5.A58 (Vddq3.3), J5.A64 (Vddq3.3), J5.B34 (Vddq3.3), J5.B40 (Vddq3.3), J5.B47 (Vddq3.3), J5.B52 (Vddq3.3), J5.B58 (Vddq3.3), J5.B64 (Vddq3.3), R23.1, R26.1, R29.1, R30.1, R31.1, R32.1, R35.1, R41.1, R46.1, R47.1, R48.1, R49.1, R50.1
- net VCC_WT is gone; now on net VCC: J23.10 (VCC), J23.14 (VCC), J23.6 (VCC)
- net GND: now also J17.S (Shield), J42.4 (GND), J13.1 (GND1), J13.2 (GND2), J13.3 (GND3), J13.4 (GND4), J13.5 (GND5); no longer J42.1 (GND)
- net PI_SCL: now also J42.2 (SCL); no longer J42.3 (SCL)
- net PI_SDA: now also J42.1 (SDA); no longer J42.4 (SDA)
- net USBHID2+: now also R122.1; no longer U17.36 (GPIO24)
- net USBHID2-: now also R123.1; no longer U17.37 (GPIO25)
- net VCC: now also C132.1, C135.1, J24.2 (5v), J24.4 (5v), J29.2 (5v), J29.4 (5v), U13.1 (IN), U13.3 (EN), U14.1 (IN), U14.3 (EN)
- net PI_3V3: now reaches J29.1 (3v3)
- net PI_3V3: now also J24.1 (3v3), J42.3 (3V3)
- net PI_BTN1: now reaches J29.11 (BCM17)
- net PI_BTN1: now also J24.11 (BCM17), J42.5 (BTN1)
- net PI_BTN2: now reaches J29.13 (BCM27)
- net PI_BTN2: now also J24.13 (BCM27), J42.6 (BTN2)
- net PI_BTN3: now reaches J29.15 (BCM22)
- net PI_BTN3: now also J24.15 (BCM22), J42.7 (BTN3)
- net PI_BTN4: now reaches J29.16 (BCM23)
- net PI_BTN4: now also J24.16 (BCM23), J42.8 (BTN4)
- net PI_BTN5: now reaches J29.7 (BCM4/GPCLK0)
- net PI_BTN5: now also J24.7 (BCM4/GPCLK0), J42.9 (BTN5)
- removed net VCC_PI: C132.1, C135.1, J24.2 (5v), J24.4 (5v), J29.2 (5v), J29.4 (5v), J42.2 (VCC), U13.1 (IN), U13.3 (EN), U14.1 (IN), U14.3 (EN)
- new net UH2+: R122.2, U17.36 (GPIO24)
- new net UH2-: R123.2, U17.37 (GPIO25)
- no-connect marks 151 -> 138
Other:
- moved on the sheet: L4
