File: kicad/opl3module/opl3module.kicad_pcb (KiCad board)
At the start: 4 copper layers, 100 x 90 mm, 143 parts, among them J1 EXT_SYNTH, J2 EXT_SYNTH, J3 EXT_SYNTH, J4 EXT_SYNTH, J5 EXT_SYNTH, J6 EXT_SYNTH, U1 YMF262, U10 YMF262, U11 YAC512, U12 TL074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

Commit message: Update Kicad project for rev.F
Parts:
- XO1, XO2, XO3, XO4, XO5, XO6: footprint llama_shared:XO_SMD5032 -> llama_shared:XO_SMD7050
- moved C10 3.00 mm to (28.7, 54.2)
- moved C18 3.00 mm to (56.7, 17.2)
- moved C2 3.00 mm to (28.7, 17.2)
- moved C26 3.00 mm to (56.7, 54.2)
- moved C34 3.00 mm to (84.7, 17.2)
- moved C42 3.00 mm to (84.7, 54.2)
- moved C1 1.73 mm to (31.5, 17.5)
- moved C17 1.73 mm to (59.5, 17.5)
- moved C33 1.73 mm to (87.5, 17.5)
- moved C25 1.73 mm to (59.5, 54.5)
- moved C41 1.73 mm to (87.5, 54.5)
- moved C9 1.73 mm to (31.5, 54.5)
Routing:
- net /YFM6_CLK: track 8.22 -> 7.01 mm
- net /YFM5_CLK: track 8.22 -> 7.01 mm
- net /YFM_CLK: track 8.22 -> 7.01 mm
- net /YFM2_CLK: track 8.22 -> 7.01 mm
- net /YFM4_CLK: track 8.22 -> 7.01 mm
- net /YFM3_CLK: track 8.22 -> 7.01 mm
- net FM5_VCC: track 30.5 -> 29.9 mm
- net FM3_VCC: track 30.5 -> 29.9 mm
Other:
- board text added: "Llama OPL3 module Revision 1.0 © 2025 Eivind Bøhler retrodreams.ca"
- board text removed: "Llama OPL3 module Revision 1.0 © 2023 Eivind Bøhler"
