File: kicad/opl3module/opl3module.kicad_sch (KiCad schematic)
At the start: 114 parts, among them J1 EXT_SYNTH, J2 EXT_SYNTH, J3 EXT_SYNTH, J4 EXT_SYNTH, J5 EXT_SYNTH, J6 EXT_SYNTH, U1 YMF262, U10 YMF262, U11 YAC512, U12 TL074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

Commit message: Update Kicad project for rev.F
Parts:
- XO1, XO2, XO3, XO4, XO5, XO6: footprint llama_shared:XO_SMD5032 -> llama_shared:XO_SMD7050; LCSC C387230 -> C41988065
